File: PCB/DiceMaster_Router/DiceMaster_Router.kicad_sch (KiCad schematic)
At the start: 34 parts, among them IC1 TPS565201DDCR, J1 RaspberryPiConnector

Commit message: Finished PCB v1
Parts:
- removed C_DBN: 100nF, symbol Device:C
- removed J_BMI270: Conn_01x06, symbol Connector_Generic:Conn_01x06
- removed Q_N2: 2N7002, symbol Transistor_FET:Q_NMOS_GSD
- removed Q_P: AO3401A, symbol Transistor_FET:Q_PMOS_GSD
- removed R_BOT, R_PD, R_SENSE, R_TOP: 10kO, symbol Device:R
- removed R_UP: 100kO, symbol Device:R
- added U1: BMI160_Breakout, Components:BMI160_Breakout, symbol BMI160:BMI160_Breakout
- C1, C3, C_OUT1, C_OUT2: footprint (none) -> Capacitor_SMD:C_0805_2012Metric
- C_BST1: renamed from C_BST; footprint (none) -> Capacitor_SMD:C_0402_1005Metric
- C_OUT3: renamed from C_OUT; footprint (none) -> Capacitor_SMD:C_0805_2012Metric
- D_FAN1: renamed from D_FAN; footprint (none) -> Diode_SMD:D_SOD-323
- IC1: footprint SOT95P280X110-6N -> Components:SOT95P280X110-6N
- J1: footprint (none) -> Connector_PinSocket_2.54mm:PinSocket_2x20_P2.54mm_Vertical
- J_A1: renamed from J_A; footprint (none) -> Connector_JST:JST_GH_SM06B-GHS-TB_1x06-1MP_P1.25mm_Horizontal
- J_B1: renamed from J_B; footprint (none) -> Connector_JST:JST_GH_SM06B-GHS-TB_1x06-1MP_P1.25mm_Horizontal
- J_BTN1: renamed from J_BTN; footprint (none) -> Connector_JST:JST_GH_SM05B-GHS-TB_1x05-1MP_P1.25mm_Horizontal
- J_C1: renamed from J_C; footprint (none) -> Connector_JST:JST_GH_SM06B-GHS-TB_1x06-1MP_P1.25mm_Horizontal
- J_D1: renamed from J_D; footprint (none) -> Connector_JST:JST_GH_SM06B-GHS-TB_1x06-1MP_P1.25mm_Horizontal
- J_E1: renamed from J_E; footprint (none) -> Connector_JST:JST_GH_SM06B-GHS-TB_1x06-1MP_P1.25mm_Horizontal
- J_F1: renamed from J_F; footprint (none) -> Connector_JST:JST_GH_SM06B-GHS-TB_1x06-1MP_P1.25mm_Horizontal
- J_FAN1: renamed from J_FAN; footprint (none) -> Connector_JST:JST_GH_SM02B-GHS-TB_1x02-1MP_P1.25mm_Horizontal
- J_SWITCH1: renamed from J_SWITCH; footprint (none) -> Connector_JST:JST_GH_SM03B-GHS-TB_1x03-1MP_P1.25mm_Horizontal
- L1: footprint (none) -> Inductor_SMD:L_Taiyo-Yuden_NR-50xx
- PiSugarPowerConnector1: renamed from PiSugarPowerConnector; footprint (none) -> Connector_JST:JST_GH_SM02B-GHS-TB_1x02-1MP_P1.25mm_Horizontal
- Q_FAN1: renamed from Q_FAN; footprint (none) -> Package_TO_SOT_SMD:SOT-23
- R_BOT1: renamed from R_BOT; value 22.1k -> 30.1k; footprint (none) -> Resistor_SMD:R_0402_1005Metric
- R_FG1: renamed from R_FG; footprint (none) -> Resistor_SMD:R_0402_1005Metric
- R_FPD1: renamed from R_FPD; footprint (none) -> Resistor_SMD:R_0402_1005Metric
- R_Top1: renamed from R_Top; footprint (none) -> Resistor_SMD:R_0402_1005Metric
Connections:
- net +5V is gone; now on net 5V_ALWAYS: PiSugarPowerConnector1.1 (Pin_1)
- net 5V_Switched is gone; now on net 5V_SWITCHED: C1.1, C3.1, D_FAN1.1 (K), IC1.3 (VIN), IC1.5 (EN), J1.2 (Pin_2), J_FAN1.1 (Pin_1)
- net +3V3: now also U1.1 (VIN)
- net BTM_4: now also J1.7 (Pin_7); no longer J1.13 (Pin_13)
- net GND: now also J1.25 (Pin_25), J1.39 (Pin_39), U1.3 (GND), U1.7 (SAO)
- net IMU_I2C_SCL: now also U1.4 (SCL)
- net IMU_I2C_SDA: now also U1.5 (SDA)
- net at R_BOT1.1, R_Top1.2: now also IC1.4 (VFB); no longer IC1.6 (VBST)
- net at C_BST1.2: now also IC1.6 (VBST); no longer IC1.4 (VFB)
- net 5V_SWITCHED: now reaches J_SWITCH1.2 (Pin_2)
- net 3V3: now reaches J1.1 (Pin_1)
- net IMU_INT2: now reaches J1.11 (Pin_11)
- net IMU_INT2: now also U1.9 (INT2)
- removed net CS: J1.12 (Pin_12), J1.24 (Pin_24), J1.27 (Pin_27), J_A1.6 (Pin_6), J_B1.6 (Pin_6), J_C1.6 (Pin_6), J_D1.6 (Pin_6), J_E1.6 (Pin_6), J_F1.6 (Pin_6)
- removed net MISO: J1.21 (Pin_21), J1.28 (Pin_28), J1.35 (Pin_35), J_A1.5 (Pin_5), J_B1.5 (Pin_5), J_C1.5 (Pin_5), J_D1.5 (Pin_5), J_E1.5 (Pin_5), J_F1.5 (Pin_5)
- removed net MOSI: J1.19 (Pin_19), J1.3 (Pin_3), J1.38 (Pin_38), J_A1.4 (Pin_4), J_B1.4 (Pin_4), J_C1.4 (Pin_4), J_D1.4 (Pin_4), J_E1.4 (Pin_4), J_F1.4 (Pin_4)
- removed net SCK: J1.23 (Pin_23), J1.40 (Pin_40), J1.5 (Pin_5), J_A1.3 (Pin_3), J_B1.3 (Pin_3), J_C1.3 (Pin_3), J_D1.3 (Pin_3), J_E1.3 (Pin_3), J_F1.3 (Pin_3)
- new net IMU_INT1: J1.13 (Pin_13), U1.10 (INT1)
- new net OCS: U1.8 (OCS)
- new net SCX: U1.11 (SCX)
- new net SDX: U1.12 (SDX)
- new net SPI_AD_CS: J1.24 (Pin_24), J_A1.6 (Pin_6), J_D1.6 (Pin_6)
- new net SPI_AD_MISO: J1.21 (Pin_21), J_A1.5 (Pin_5), J_D1.5 (Pin_5)
- new net SPI_AD_MOSI: J1.19 (Pin_19), J_A1.4 (Pin_4), J_D1.4 (Pin_4)
- new net SPI_AD_SCL: J1.23 (Pin_23), J_A1.3 (Pin_3), J_D1.3 (Pin_3)
- new net SPI_BE_CS: J1.12 (Pin_12), J_B1.6 (Pin_6), J_E1.6 (Pin_6)
- new net SPI_BE_MISO: J1.35 (Pin_35), J_B1.5 (Pin_5), J_E1.5 (Pin_5)
- new net SPI_BE_MOSI: J1.38 (Pin_38), J_B1.4 (Pin_4), J_E1.4 (Pin_4)
- new net SPI_BE_SCL: J1.40 (Pin_40), J_B1.3 (Pin_3), J_E1.3 (Pin_3)
- new net SPI_CF_CS: J1.27 (Pin_27), J_C1.6 (Pin_6), J_F1.6 (Pin_6)
- new net SPI_CF_MISO: J1.28 (Pin_28), J_C1.5 (Pin_5), J_F1.5 (Pin_5)
- new net SPI_CF_MOSI: J1.3 (Pin_3), J_C1.4 (Pin_4), J_F1.4 (Pin_4)
- new net SPI_CF_SCL: J1.5 (Pin_5), J_C1.3 (Pin_3), J_F1.3 (Pin_3)
- no-connect marks 0 -> 22
Other:
- moved on the sheet: C_BST1, J_FAN1, PiSugarPowerConnector1
