File: PCB/DiceMaster_Router/DiceMaster_Router.kicad_pcb (KiCad board)
At the start: 2 copper layers, 60 x 60 mm, 26 parts, among them IC1 TPS565201DDCR, J1 RaspberryPiConnector, U1 BMI160_Breakout

Commit message: finalized pcb v1 for prod
Parts:
- J_SWITCH1: value SW -> J_SW
- PiSugarPowerConnector1: value Battery -> J_BAT
Other:
- board text added: "J_B1"
- board text added: "J_C1"
- board text added: "J_FAN"
Changed lines of the file:
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@@
 			(outputformat 1)
 			(mirror no)
-			(drillshape 1)
+			(drillshape 0)
 			(scaleselection 1)
-			(outputdirectory "")
+			(outputdirectory "gerbers/")
 		)
 	)
@@
 			(at 5 -10 0)
 			(layer "F.SilkS")
+			(hide yes)
 			(effects
 				(font
@@
 		)
 		(property "Value" "BMI160_Breakout"
-			(at -0.5 11.5 0)
+			(at 2.5 6.5 0)
 			(layer "F.Fab")
 			(effects
@@
 			(layer "F.CrtYd")
 		)
-		(fp_text user "Pin 1"
+		(fp_text user "IMU"
 			(at 1.5 0 0)
 			(layer "F.SilkS")
@@
 		(tags "connector JST GH horizontal")
 		(property "Reference" "J_A1"
-			(at 0 -4 0)
+			(at 5.5 -3 0)
 			(layer "F.SilkS")
 			(effects
@@
 		(tags "connector JST GH horizontal")
 		(property "Reference" "J_F1"
-			(at 5.625 -2.65 90)
+			(at 4.625 -3.65 0)
 			(layer "F.SilkS")
 			(effects
@@
 			(at 2.525 0.35 90)
 			(layer "F.SilkS")
+			(hide yes)
 			(effects
 				(font
@@
 			(at 2 1 90)
 			(layer "F.SilkS")
+			(hide yes)
 			(effects
 				(font
@@
 		(tags "connector JST GH horizontal")
 		(property "Reference" "J_E1"
-			(at 3.125 -4.35 90)
+			(at -4.875 -3.85 0)
 			(layer "F.SilkS")
 			(effects
@@
 		(tags "connector JST GH horizontal")
 		(property "Reference" "J_D1"
-			(at 0 -3.9 0)
+			(at -2 4.35 0)
 			(layer "F.SilkS")
 			(effects
@@
 			)
 		)
-		(property "Value" "SW"
+		(property "Value" "J_SW"
 			(at -3 4 0)
 			(layer "F.SilkS")
@@
 			)
 		)
-		(property "Value" "Battery"
-			(at -2.475 3.85 0)
+		(property "Value" "J_BAT"
+			(at -2.975 3.85 0)
 			(layer "F.SilkS")
 			(effects
@@
 		(layer "Edge.Cuts")
 	)
+	(gr_text "J_B1"
+		(at 59 85 0)
+		(layer "F.SilkS")
+		(effects
+			(font
+				(size 1 1)
+				(thickness 0.1)
+			)
+			(justify left bottom)
+		)
+	)
+	(gr_text "J_C1"
+		(at 59 98.46 0)
+		(layer "F.SilkS")
+		(effects
+			(font
+				(size 1 1)
+				(thickness 0.1)
+			)
+			(justify left bottom)
+		)
+	)
+	(gr_text "J_FAN"
+		(at 102.5 55 0)
+		(layer "F.SilkS")
+		(effects
+			(font
+				(size 1 1)
+				(thickness 0.1)
+			)
+			(justify left bottom)
+		)
+	)
 	(segment
